Commit message: update

File: urdf/so101_new_calib.urdf (robot description, URDF)
Before this commit: robot so101_new_calib, 8 links, 7 joints
Joints:
- added joint camera_joint: type fixed, parent wrist_roll_follower, child camera_link, origin xyz=0 0 0.04 rpy=0 1.5708 0

File: urdf/so_arm101_camera.urdf (robot description, URDF)
Before this commit: robot so_arm101_camera, 8 links, 7 joints
Links:
- link base_link: geometry collision cylinder length=0.05 radius=0.06; visual mesh filename=assets/base_so101_v2.stl
- link motor_holder_base: geometry collision cylinder length=0.04 radius=0.04; visual mesh filename=assets/motor_holder_so101_base_v1.stl
- link rotation_pitch: geometry collision cylinder length=0.06 radius=0.025; visual mesh filename=assets/rotation_pitch_so101_v1.stl
- link under_arm: geometry collision box size=0.08 0.04 0.1; visual mesh filename=assets/under_arm_so101_v1.stl
- link upper_arm: geometry collision box size=0.06 0.04 0.15; visual mesh filename=assets/upper_arm_so101_v1.stl
- link wrist_roll_follower: geometry collision cylinder length=0.04 radius=0.015; visual mesh filename=assets/wrist_roll_follower_so101_v1.stl
- link wrist_roll_pitch: geometry collision cylinder length=0.05 radius=0.02; visual mesh filename=assets/wrist_roll_pitch_so101_v2.stl

Commit message: URDF, Camera fixed

File: urdf/so101_new_calib.urdf (robot description, URDF)
Before this commit: robot so101_new_calib, 8 links, 7 joints
Links:
- added link camera_link, mass 0.01; collision box size=0.03 0.03 0.02; visual box size=0.03 0.03 0.02
Joints:
- added joint camera_joint: type fixed, parent gripper_frame_link, child camera_link, origin xyz=0 0 0.02 rpy=0 -1.5708 0
